Commit message: Add files via upload

File: final_description/urdf/final.xacro (robot description, xacro)
@@ -6,5 +6,5 @@
 <link name="base_link">
   <inertial>
-    <origin xyz="-0.021518218467853914 0.23351950797477217 0.23670607205875357" rpy="0 0 0"/>
+    <origin xyz="-0.04025794040578778 0.14165010590483765 0.2860735834847339" rpy="0 0 0"/>
     <mass value="17.97264000000002"/>
     <inertia ixx="1.833137" iyy="1.542102" izz="1.955592" ixy="0.030245" iyz="-0.287683" ixz="0.030749"/>
@@ -13,5 +13,5 @@
     <origin xyz="0 0 0" rpy="0 0 0"/>
     <geometry>
-      <mesh filename="package://final_description/meshes/base_link.stl" scale="0.001 0.001 0.001"/>
+      <mesh filename="file://$(find final_description)/meshes/base_link.stl" scale="0.001 0.001 0.001"/>
     </geometry>
     <material name="silver"/>
@@ -20,5 +20,5 @@
     <origin xyz="0 0 0" rpy="0 0 0"/>
     <geometry>
-      <mesh filename="package://final_description/meshes/base_link.stl" scale="0.001 0.001 0.001"/>
+      <mesh filename="file://$(find final_description)/meshes/base_link.stl" scale="0.001 0.001 0.001"/>
     </geometry>
   </collision>
@@ -26,19 +26,19 @@
 <link name="foundation__base_1">
   <inertial>
-    <origin xyz="-0.005187232824595431 -0.00018279822615355212 0.2337928136509641" rpy="0 0 0"/>
+    <origin xyz="0.01355204523747059 0.09168679970391208 0.18442532507694448" rpy="0 0 0"/>
     <mass value="920.4727092380529"/>
     <inertia ixx="48.985183" iyy="41.31025" izz="48.576431" ixy="0.000622" iyz="0.048602" ixz="-0.042143"/>
   </inertial>
   <visual>
-    <origin xyz="-0.006599 0.217347 -0.001287" rpy="0 0 0"/>
+    <origin xyz="0.03088 0.401086 -0.100022" rpy="0 0 0"/>
     <geometry>
-      <mesh filename="package://final_description/meshes/foundation__base_1.stl" scale="0.001 0.001 0.001"/>
+      <mesh filename="file://$(find final_description)/meshes/foundation__base_1.stl" scale="0.001 0.001 0.001"/>
     </geometry>
     <material name="silver"/>
   </visual>
   <collision>
-    <origin xyz="-0.006599 0.217347 -0.001287" rpy="0 0 0"/>
+    <origin xyz="0.03088 0.401086 -0.100022" rpy="0 0 0"/>
     <geometry>
-      <mesh filename="package://final_description/meshes/foundation__base_1.stl" scale="0.001 0.001 0.001"/>
+      <mesh filename="file://$(find final_description)/meshes/foundation__base_1.stl" scale="0.001 0.001 0.001"/>
     </geometry>
   </collision>
@@ -46,19 +46,19 @@
 <link name="foundation_fork_1">
   <inertial>
-    <origin xyz="-0.004766196492609534 0.18491027281057554 -0.004542791939917135" rpy="0 0 0"/>
+    <origin xyz="0.013060697203541947 0.27683187305279844 -0.05391028051391977" rpy="0 0 0"/>
     <mass value="2.0983050311927904"/>
-    <inertia ixx="0.018488" iyy="0.020902" izz="0.024893" ixy="8.8e-05" iyz="0.001405" ixz="5.5e-05"/>
+    <inertia ixx="0.018494" iyy="0.020896" izz="0.024893" ixy="0.000153" iyz="0.001403" ixz="9.3e-05"/>
   </inertial>
   <visual>
-    <origin xyz="-0.006599 0.287347 -0.692287" rpy="0 0 0"/>
+    <origin xyz="0.03088 0.471086 -0.791022" rpy="0 0 0"/>
     <geometry>
-      <mesh filename="package://final_description/meshes/foundation_fork_1.stl" scale="0.001 0.001 0.001"/>
+      <mesh filename="file://$(find final_description)/meshes/foundation_fork_1.stl" scale="0.001 0.001 0.001"/>
     </geometry>
     <material name="silver"/>
   </visual>
   <collision>
-    <origin xyz="-0.006599 0.287347 -0.692287" rpy="0 0 0"/>
+    <origin xyz="0.03088 0.471086 -0.791022" rpy="0 0 0"/>
     <geometry>
-      <mesh filename="package://final_description/meshes/foundation_fork_1.stl" scale="0.001 0.001 0.001"/>
+      <mesh filename="file://$(find final_description)/meshes/foundation_fork_1.stl" scale="0.001 0.001 0.001"/>
     </geometry>
   </collision>
@@ -66,19 +66,19 @@
 <link name="hand_fork_1">
   <inertial>
-    <origin xyz="-1.029072678544643 -0.1359581722157417 0.09150144060797305" rpy="0 0 0"/>
+    <origin xyz="-1.1013898197968075 0.006896777757352757 0.04959859992152271" rpy="0 0 0"/>
     <mass value="0.19515039122298017"/>
-    <inertia ixx="0.000118" iyy="0.000413" izz="0.000452" ixy="1.2e-05" iyz="1.6e-05" ixz="1e-06"/>
+    <inertia ixx="0.000118" iyy="0.000412" izz="0.000452" ixy="2e-05" iyz="1.6e-05" ixz="2e-06"/>
   </inertial>
   <visual>
-    <origin xyz="-1.055408 -0.79118 -0.902226" rpy="0 0 0"/>
+    <origin xyz="-1.126841 -0.530578 -1.020832" rpy="0 0 0"/>
     <geometry>
-      <mesh filename="package://final_description/meshes/hand_fork_1.stl" scale="0.001 0.001 0.001"/>
+      <mesh filename="file://$(find final_description)/meshes/hand_fork_1.stl" scale="0.001 0.001 0.001"/>
     </geometry>
     <material name="silver"/>
   </visual>
   <collision>
-    <origin xyz="-1.055408 -0.79118 -0.902226" rpy="0 0 0"/>
+    <origin xyz="-1.126841 -0.530578 -1.020832" rpy="0 0 0"/>
     <geometry>
-      <mesh filename="package://final_description/meshes/hand_fork_1.stl" scale="0.001 0.001 0.001"/>
+      <mesh filename="file://$(find final_description)/meshes/hand_fork_1.stl" scale="0.001 0.001 0.001"/>
     </geometry>
   </collision>
@@ -86,19 +86,19 @@
 <link name="hand_1">
   <inertial>
-    <origin xyz="1.0622973829575801 0.5189730926582943 0.4557263448303449" rpy="0 0 0"/>
+    <origin xyz="1.1443603093404926 0.36632887796131397 0.40450650414389033" rpy="0 0 0"/>
     <mass value="0.39288844288416375"/>
-    <inertia ixx="0.008983" iyy="0.001945" izz="0.008227" ixy="-0.000291" iyz="0.002948" ixz="0.000122"/>
+    <inertia ixx="0.008963" iyy="0.001966" izz="0.008227" ixy="-0.000481" iyz="0.002943" ixz="0.000201"/>
   </inertial>
   <visual>
-    <origin xyz="1.049329 0.187612 -0.662019" rpy="0 0 0"/>
+    <origin xyz="1.141028 0.152235 -0.789942" rpy="0 0 0"/>
     <geometry>
-      <mesh filename="package://final_description/meshes/hand_1.stl" scale="0.001 0.001 0.001"/>
+      <mesh filename="file://$(find final_description)/meshes/hand_1.stl" scale="0.001 0.001 0.001"/>
     </geometry>
     <material name="silver"/>
   </visual>
   <collision>
-    <origin xyz="1.049329 0.187612 -0.662019" rpy="0 0 0"/>
+    <origin xyz="1.141028 0.152235 -0.789942" rpy="0 0 0"/>
     <geometry>
-      <mesh filename="package://final_description/meshes/hand_1.stl" scale="0.001 0.001 0.001"/>
+      <mesh filename="file://$(find final_description)/meshes/hand_1.stl" scale="0.001 0.001 0.001"/>
     </geometry>
   </collision>
@@ -106,19 +106,19 @@
 <link name="end_effector_1">
   <inertial>
-    <origin xyz="0.02998999546059815 0.07686702308209326 -0.1674246665384953" rpy="0 0 0"/>
+    <origin xyz="0.03877631864976241 0.17128922609145047 -0.06320835446115469" rpy="0 0 0"/>
     <mass value="0.5354810781353961"/>
-    <inertia ixx="0.003599" iyy="0.00302" izz="0.000874" ixy="-1.3e-05" iyz="0.001278" ixz="2.9e-05"/>
+    <inertia ixx="0.003588" iyy="0.000679" izz="0.003225" ixy="-0.000178" iyz="0.001071" ixz="6.6e-05"/>
   </inertial>
   <visual>
-    <origin xyz="-0.002351 -0.680353 -0.98499" rpy="0 0 0"/>
+    <origin xyz="-0.002155 -0.563245 -1.061693" rpy="0 0 0"/>
     <geometry>
-      <mesh filename="package://final_description/meshes/end_effector_1.stl" scale="0.001 0.001 0.001"/>
+      <mesh filename="file://$(find final_description)/meshes/end_effector_1.stl" scale="0.001 0.001 0.001"/>
     </geometry>
     <material name="silver"/>
   </visual>
   <collision>
-    <origin xyz="-0.002351 -0.680353 -0.98499" rpy="0 0 0"/>
+    <origin xyz="-0.002155 -0.563245 -1.061693" rpy="0 0 0"/>
     <geometry>
-      <mesh filename="package://final_description/meshes/end_effector_1.stl" scale="0.001 0.001 0.001"/>
+      <mesh filename="file://$(find final_description)/meshes/end_effector_1.stl" scale="0.001 0.001 0.001"/>
     </geometry>
   </collision>
@@ -126,24 +126,24 @@
 <link name="forearm_1">
   <inertial>
-    <origin xyz="-0.08998662668791652 -0.025200150523567236 -0.6179977746399161" rpy="0 0 0"/>
+    <origin xyz="-0.11185843293812174 -0.11465010627249536 -0.6640390159850146" rpy="0 0 0"/>
     <mass value="1.1580779637924898"/>
-    <inertia ixx="0.03619" iyy="0.025639" izz="0.031664" ixy="-0.000436" iyz="-0.017312" ixz="-0.000715"/>
+    <inertia ixx="0.036173" iyy="0.028711" izz="0.028609" ixy="-0.000513" iyz="-0.017547" ixz="-0.0012"/>
   </inertial>
   <visual>
-    <origin xyz="-0.089923 0.003711 -1.516287" rpy="0 0 0"/>
+    <origin xyz="-0.093927 0.009043 -1.615022" rpy="0 0 0"/>
     <geometry>
-      <mesh filename="package://final_description/meshes/forearm_1.stl" scale="0.001 0.001 0.001"/>
+      <mesh filename="file://$(find final_description)/meshes/forearm_1.stl" scale="0.001 0.001 0.001"/>
     </geometry>
     <material name="silver"/>
   </visual>
   <collision>
-    <origin xyz="-0.089923 0.003711 -1.516287" rpy="0 0 0"/>
+    <origin xyz="-0.093927 0.009043 -1.615022" rpy="0 0 0"/>
     <geometry>
-      <mesh filename="package://final_description/meshes/forearm_1.stl" scale="0.001 0.001 0.001"/>
+      <mesh filename="file://$(find final_description)/meshes/forearm_1.stl" scale="0.001 0.001 0.001"/>
     </geometry>
   </collision>
 </link>
 <joint name="rigid_1" type="fixed">
-  <origin xyz="0.006599 -0.217347 0.001287" rpy="0 0 0"/>
+  <origin xyz="-0.03088 -0.401086 0.100022" rpy="0 0 0"/>
   <parent link="base_link"/>
   <child link="foundation__base_1"/>
@@ -156,29 +156,29 @@
 </joint>
 <joint name="hand_fork" type="revolute">
-  <origin xyz="2.104737 0.978792 0.240207" rpy="0 0 0"/>
+  <origin xyz="2.267869 0.682813 0.23089" rpy="0 0 0"/>
   <parent link="hand_1"/>
   <child link="hand_fork_1"/>
-  <axis xyz="-0.038751 -0.938893 0.34202"/>
+  <axis xyz="-0.064124 -0.937502 0.34202"/>
   <limit upper="0.0" lower="-3.141593" effort="100" velocity="100"/>
 </joint>
 <joint name="hand_forearm" type="revolute">
-  <origin xyz="-1.139252 -0.183901 -0.854268" rpy="0 0 0"/>
+  <origin xyz="-1.234955 -0.143192 -0.82508" rpy="0 0 0"/>
   <parent link="forearm_1"/>
   <child link="hand_1"/>
-  <axis xyz="-0.999149 0.041238 -0.0"/>
+  <axis xyz="-0.997669 0.068239 0.0"/>
   <limit upper="2.268928" lower="0.872665" effort="100" velocity="100"/>
 </joint>
 <joint name="end_fork" type="revolute">
-  <origin xyz="-1.053057 -0.110827 0.082764" rpy="0 0 0"/>
+  <origin xyz="-1.124686 0.032667 0.040861" rpy="0 0 0"/>
   <parent link="hand_fork_1"/>
   <child link="end_effector_1"/>
-  <axis xyz="0.999126 -0.041768 -0.001458"/>
+  <axis xyz="0.997632 -0.068768 -0.001458"/>
   <limit upper="1.570796" lower="-1.570796" effort="100" velocity="100"/>
 </joint>
 <joint name="forearm_fork" type="revolute">
-  <origin xyz="0.083324 0.283636 0.824" rpy="0 0 0"/>
+  <origin xyz="0.124807 0.462043 0.824" rpy="0 0 0"/>
   <parent link="foundation_fork_1"/>
   <child link="forearm_1"/>
-  <axis xyz="0.999149 -0.041238 0.0"/>
+  <axis xyz="0.997669 -0.068239 -0.0"/>
   <limit upper="-0.523599" lower="-2.094395" effort="100" velocity="100"/>
 </joint>

Commit message: Add files via upload

File: final_description/urdf/final.xacro (robot description, xacro)
@@ -155,31 +155,27 @@
   <axis xyz="-0.0 -0.0 1.0"/>
 </joint>
-<joint name="hand_fork" type="revolute">
+<joint name="hand_fork" type="continuous">
   <origin xyz="2.267869 0.682813 0.23089" rpy="0 0 0"/>
   <parent link="hand_1"/>
   <child link="hand_fork_1"/>
   <axis xyz="-0.064124 -0.937502 0.34202"/>
-  <limit upper="0.0" lower="-3.141593" effort="100" velocity="100"/>
 </joint>
-<joint name="hand_forearm" type="revolute">
+<joint name="hand_forearm" type="continuous">
   <origin xyz="-1.234955 -0.143192 -0.82508" rpy="0 0 0"/>
   <parent link="forearm_1"/>
   <child link="hand_1"/>
   <axis xyz="-0.997669 0.068239 0.0"/>
-  <limit upper="2.268928" lower="0.872665" effort="100" velocity="100"/>
 </joint>
-<joint name="end_fork" type="revolute">
+<joint name="end_fork" type="continuous">
   <origin xyz="-1.124686 0.032667 0.040861" rpy="0 0 0"/>
   <parent link="hand_fork_1"/>
   <child link="end_effector_1"/>
   <axis xyz="0.997632 -0.068768 -0.001458"/>
-  <limit upper="1.570796" lower="-1.570796" effort="100" velocity="100"/>
 </joint>
-<joint name="forearm_fork" type="revolute">
+<joint name="forearm_fork" type="continuous">
   <origin xyz="0.124807 0.462043 0.824" rpy="0 0 0"/>
   <parent link="foundation_fork_1"/>
   <child link="forearm_1"/>
   <axis xyz="0.997669 -0.068239 -0.0"/>
-  <limit upper="-0.523599" lower="-2.094395" effort="100" velocity="100"/>
 </joint>
 </robot>
